Commit message: Update brick housing inertia

File: urdf/base_macros/brick_housing.urdf.xacro (robot description, xacro)
@@ -74,14 +74,14 @@
             <xacro:if value="${with_wheel}">
                 <inertial>
-                    <mass value="4.554" />
-                    <origin xyz="0.00005 0.00009 0.12048" />
-                    <inertia  ixx="0.0512" ixy="0.0000062" ixz="0.0000224" iyy="0.051012" iyz="0.000027" izz="0.062741" />
+                    <mass value="9.6933" />
+                    <origin xyz="0.00026 0.00510 0.07547" rpy="0 0 0"/>
+                    <inertia ixx="0.08383681353" ixy="0.00004888825" ixz="0.00013579563" iyy="0.08722388730" iyz="-0.00202543540" izz="0.07461687470" />
                 </inertial>
             </xacro:if>
             <xacro:unless value="${with_wheel}">
                 <inertial>
-                    <mass value="4.554" />
-                    <origin xyz="0.00005 0.00009 0.12048" />
-                    <inertia  ixx="0.0512" ixy="0.0000062" ixz="0.0000224" iyy="0.051012" iyz="0.000027" izz="0.062741" />
+                    <mass value="4.6706"/>
+                    <origin xyz="0.00026 0.00074 0.12235" rpy="0 0 0"/>
+                    <inertia ixx="0.05201415149" ixy="0.00003134654" ixz="0.00009162302" iyy="0.05172495462" iyz="0.00024791202" izz="0.06298895653"/>
                 </inertial>
 		    </xacro:unless>
