Commit message: Update kelo drive inertia

File: urdf/base_macros/kelo_drive.urdf.xacro (robot description, xacro)
@@ -74,6 +74,9 @@
                 </geometry>
             </collision>
-            <!--TODO: Set the correct inertia-->
-            <xacro:cuboid_inertia mass="10.0" length="0.233" breadth="0.233" height="0.233"/>
+            <inertial>
+                <origin xyz="0.00023 -0.00095 0.04843" rpy="0 0 0"/>
+                <mass value="1.46273"/>
+                <inertia ixx="0.00302046423" ixy="0.00000851844" ixz="0.00001188180" iyy="0.00326495472" iyz="0.00001855408" izz="0.00386072964"/>
+            </inertial>
         </link>
         <!-- LEFT HUB WHEEL -->

File: urdf/base_macros/kelo_drive_wheel.urdf.xacro (robot description, xacro)
@@ -71,14 +71,9 @@
                 </geometry>
             </collision>
-            <!-- xacro:cylinder_inertia mass="0.5" radius="0.0515" length="0.035" center_of_mass_roll="1.570796327"/ -->
-<!--
             <inertial>
-                <mass value="2.0829" />
-                <origin xyz="0 0.00038 -0.00002" />
-                <inertia  ixx="0.001385" ixy="0" ixz="0" iyy="0.001998" iyz="-0.0000005" izz="0.0013857" />
+                <origin xyz="0 0 0" rpy="0 0 0"/>
+                <mass value="1.56317"/>
+                <inertia ixx="0.00101253363" ixy="0.00000000000" ixz="0.00000001020" iyy="0.00157998524" iyz="-0.00000055474" izz="0.00101282739"/>
             </inertial>
--->
-            <!--HACK: Use large cuboid inertias to fix the issue that the model breaks when JointVelocity controller is activated -->
-            <xacro:cuboid_inertia mass="10.0" length="0.233" breadth="0.233" height="0.233"/>
         </link>
     </xacro:macro>

Commit message: Add new top part link to kelo drive

File: urdf/base_macros/kelo_drive.urdf.xacro (robot description, xacro)
@@ -80,4 +80,31 @@
             </inertial>
         </link>
+        <link name="${name}_drive_top_part_link">
+            <visual>
+                <origin xyz="0 0 0" rpy="0 0 0"/>
+                <geometry>
+                    <mesh filename="file://$(find robile_description)/meshes/kelo_drive/kelo_drive_top_part.dae" scale="1 1 1"/>
+                </geometry>
+                <material name="black">
+                    <color rgba="0.0 0.0 0.0 1.0"/>
+                </material>
+            </visual>
+            <collision>
+                <origin xyz="0 0 0" rpy="0 0 0"/>
+                <geometry>
+                    <mesh filename="file://$(find robile_description)/meshes/kelo_drive/kelo_drive_top_part.dae" scale="1 1 1"/>
+                </geometry>
+            </collision>
+            <inertial>
+                <origin xyz="0.00054 -0.00146 0.01031" rpy="0 0 0"/>
+                <mass value="0.43207"/>
+                <inertia ixx="0.00036965278" ixy="0.00001352474" ixz="-0.00000005992" iyy="0.00039670119" iyz="0.00000019355" izz="0.00073957435"/>
+            </inertial>
+        </link>
+        <joint name="${name}_drive_top_part_joint" type="fixed">
+            <origin xyz="0 0 0.09" rpy="0 0 0"/>
+            <parent link="${parent}"/>
+            <child link="${name}_drive_top_part_link"/>
+        </joint>
         <!-- LEFT HUB WHEEL -->
         <xacro:kelo_drive_wheel name="${name}_left_hub_wheel" parent="${name}_pivot_link" movable_joints="${movable_joints}">

Commit message: Add joint limits to pivot joint in kelo drive

File: urdf/base_macros/kelo_drive.urdf.xacro (robot description, xacro)
@@ -38,4 +38,5 @@
             <parent link="${parent}"/>
             <child link="${name}_pivot_link" />
+            <limit effort="10.0" velocity="10.0"/>
         </joint>
         <transmission name="${name}_pivot_transmission">
