Commit message: Add use_real_inertia flag

File: robots/2_wheel_config.urdf.xacro (robot description, xacro)
@@ -31,4 +31,5 @@
 <robot xmlns:xacro="http://ros.org/wiki/xacro" name="2_wheel_config" >
     <xacro:arg name="movable_joints" default="true"/>
+    <xacro:arg name="use_real_inertia" default="false"/>
     <!-- Include desired robile bricks -->
     <xacro:include filename="$(find robile_description)/urdf/robile_bricks/robile_active_wheel_brick.urdf.xacro" />
@@ -50,8 +51,8 @@
         <origin xyz="0.0 -0.1165 0.05" rpy="0.0 0.0 0.0"/>
     </xacro:robile_master_battery_brick>
-    <xacro:robile_active_wheel_brick name="robile_5" parent="base_link" movable_joints="$(arg movable_joints)">
+    <xacro:robile_active_wheel_brick name="robile_5" parent="base_link" movable_joints="$(arg movable_joints)" use_real_inertia="$(arg use_real_inertia)">
         <origin xyz="-0.233 0.1165 0.05" rpy="0.0 0.0 0.0"/>
     </xacro:robile_active_wheel_brick>
-    <xacro:robile_active_wheel_brick name="robile_6" parent="base_link" movable_joints="$(arg movable_joints)">
+    <xacro:robile_active_wheel_brick name="robile_6" parent="base_link" movable_joints="$(arg movable_joints)" use_real_inertia="$(arg use_real_inertia)">
         <origin xyz="-0.233 -0.1165 0.05" rpy="0.0 0.0 0.0"/>
     </xacro:robile_active_wheel_brick>

File: robots/4_wheel_config.urdf.xacro (robot description, xacro)
@@ -31,4 +31,5 @@
 <robot xmlns:xacro="http://ros.org/wiki/xacro" name="4_wheel_config" >
     <xacro:arg name="movable_joints" default="true"/>
+    <xacro:arg name="use_real_inertia" default="false"/>
     <!-- Include desired robile bricks -->
     <xacro:include filename="$(find robile_description)/urdf/robile_bricks/robile_active_wheel_brick.urdf.xacro" />
@@ -37,8 +38,8 @@
     <link name="base_link"/>
     <!-- Build platform using robile bricks -->
-    <xacro:robile_active_wheel_brick name="robile_1" parent="base_link" movable_joints="$(arg movable_joints)">
+    <xacro:robile_active_wheel_brick name="robile_1" parent="base_link" movable_joints="$(arg movable_joints)" use_real_inertia="$(arg use_real_inertia)">
         <origin xyz="0.233 0.1165 0.05" rpy="0.0 0.0 0.0"/>
     </xacro:robile_active_wheel_brick>
-    <xacro:robile_active_wheel_brick name="robile_2" parent="base_link" movable_joints="$(arg movable_joints)">
+    <xacro:robile_active_wheel_brick name="robile_2" parent="base_link" movable_joints="$(arg movable_joints)" use_real_inertia="$(arg use_real_inertia)">
         <origin xyz="0.233 -0.1165 0.05" rpy="0.0 0.0 0.0"/>
     </xacro:robile_active_wheel_brick>
@@ -49,8 +50,8 @@
         <origin xyz="0.0 -0.1165 0.05" rpy="0.0 0.0 0.0"/>
     </xacro:robile_master_battery_brick>
-    <xacro:robile_active_wheel_brick name="robile_5" parent="base_link" movable_joints="$(arg movable_joints)">
+    <xacro:robile_active_wheel_brick name="robile_5" parent="base_link" movable_joints="$(arg movable_joints)" use_real_inertia="$(arg use_real_inertia)">
         <origin xyz="-0.233 0.1165 0.05" rpy="0.0 0.0 0.0"/>
     </xacro:robile_active_wheel_brick>
-    <xacro:robile_active_wheel_brick name="robile_6" parent="base_link" movable_joints="$(arg movable_joints)">
+    <xacro:robile_active_wheel_brick name="robile_6" parent="base_link" movable_joints="$(arg movable_joints)" use_real_inertia="$(arg use_real_inertia)">
         <origin xyz="-0.233 -0.1165 0.05" rpy="0.0 0.0 0.0"/>
     </xacro:robile_active_wheel_brick>

File: robots/4_wheel_double_microscan_config.urdf.xacro (robot description, xacro)
@@ -32,4 +32,5 @@
 <robot xmlns:xacro="http://ros.org/wiki/xacro" name="4_wheel_double_microscan_config" >
     <xacro:arg name="movable_joints" default="true"/>
+    <xacro:arg name="use_real_inertia" default="false"/>
     <!-- Include desired robile bricks -->
     <xacro:include filename="$(find robile_description)/urdf/robile_bricks/robile_active_wheel_brick.urdf.xacro" />
@@ -39,8 +40,8 @@
     <link name="base_link"/>
     <!-- Build platform using robile bricks -->
-    <xacro:robile_active_wheel_brick name="robile_1" parent="base_link" movable_joints="$(arg movable_joints)">
+    <xacro:robile_active_wheel_brick name="robile_1" parent="base_link" movable_joints="$(arg movable_joints)" use_real_inertia="$(arg use_real_inertia)">
         <origin xyz="0.233 0.1165 0.05" rpy="0.0 0.0 0.0"/>
     </xacro:robile_active_wheel_brick>
-    <xacro:robile_active_wheel_brick name="robile_2" parent="base_link" movable_joints="$(arg movable_joints)">
+    <xacro:robile_active_wheel_brick name="robile_2" parent="base_link" movable_joints="$(arg movable_joints)" use_real_inertia="$(arg use_real_inertia)">
         <origin xyz="0.233 -0.1165 0.05" rpy="0.0 0.0 0.0"/>
     </xacro:robile_active_wheel_brick>
@@ -51,8 +52,8 @@
         <origin xyz="0.0 -0.1165 0.05" rpy="0.0 0.0 0.0"/>
     </xacro:robile_master_battery_brick>
-    <xacro:robile_active_wheel_brick name="robile_5" parent="base_link" movable_joints="$(arg movable_joints)">
+    <xacro:robile_active_wheel_brick name="robile_5" parent="base_link" movable_joints="$(arg movable_joints)" use_real_inertia="$(arg use_real_inertia)">
         <origin xyz="-0.233 0.1165 0.05" rpy="0.0 0.0 0.0"/>
     </xacro:robile_active_wheel_brick>
-    <xacro:robile_active_wheel_brick name="robile_6" parent="base_link" movable_joints="$(arg movable_joints)">
+    <xacro:robile_active_wheel_brick name="robile_6" parent="base_link" movable_joints="$(arg movable_joints)" use_real_inertia="$(arg use_real_inertia)">
         <origin xyz="-0.233 -0.1165 0.05" rpy="0.0 0.0 0.0"/>
     </xacro:robile_active_wheel_brick>

File: robots/4_wheel_double_uam_config.urdf.xacro (robot description, xacro)
@@ -32,4 +32,5 @@
 <robot xmlns:xacro="http://ros.org/wiki/xacro" name="4_wheel_double_microscan_config" >
     <xacro:arg name="movable_joints" default="true"/>
+    <xacro:arg name="use_real_inertia" default="false"/>
     <!-- Include desired robile bricks -->
     <xacro:include filename="$(find robile_description)/urdf/robile_bricks/robile_active_wheel_brick.urdf.xacro" />
@@ -39,8 +40,8 @@
     <link name="base_link"/>
     <!-- Build platform using robile bricks -->
-    <xacro:robile_active_wheel_brick name="robile_1" parent="base_link" movable_joints="$(arg movable_joints)">
+    <xacro:robile_active_wheel_brick name="robile_1" parent="base_link" movable_joints="$(arg movable_joints)" use_real_inertia="$(arg use_real_inertia)">
         <origin xyz="0.233 0.1165 0.05" rpy="0.0 0.0 0.0"/>
     </xacro:robile_active_wheel_brick>
-    <xacro:robile_active_wheel_brick name="robile_2" parent="base_link" movable_joints="$(arg movable_joints)">
+    <xacro:robile_active_wheel_brick name="robile_2" parent="base_link" movable_joints="$(arg movable_joints)" use_real_inertia="$(arg use_real_inertia)">
         <origin xyz="0.233 -0.1165 0.05" rpy="0.0 0.0 0.0"/>
     </xacro:robile_active_wheel_brick>
@@ -51,8 +52,8 @@
         <origin xyz="0.0 -0.1165 0.05" rpy="0.0 0.0 0.0"/>
     </xacro:robile_master_battery_brick>
-    <xacro:robile_active_wheel_brick name="robile_5" parent="base_link" movable_joints="$(arg movable_joints)">
+    <xacro:robile_active_wheel_brick name="robile_5" parent="base_link" movable_joints="$(arg movable_joints)" use_real_inertia="$(arg use_real_inertia)">
         <origin xyz="-0.233 0.1165 0.05" rpy="0.0 0.0 0.0"/>
     </xacro:robile_active_wheel_brick>
-    <xacro:robile_active_wheel_brick name="robile_6" parent="base_link" movable_joints="$(arg movable_joints)">
+    <xacro:robile_active_wheel_brick name="robile_6" parent="base_link" movable_joints="$(arg movable_joints)" use_real_inertia="$(arg use_real_inertia)">
         <origin xyz="-0.233 -0.1165 0.05" rpy="0.0 0.0 0.0"/>
     </xacro:robile_active_wheel_brick>

File: robots/4_wheel_lidar_config.urdf.xacro (robot description, xacro)
@@ -32,4 +32,5 @@
 <robot xmlns:xacro="http://ros.org/wiki/xacro" name="4_wheel_lidar_config" >
     <xacro:arg name="movable_joints" default="true"/>
+    <xacro:arg name="use_real_inertia" default="false"/>
     <!-- Include desired robile bricks -->
     <xacro:include filename="$(find robile_description)/urdf/robile_bricks/robile_active_wheel_brick.urdf.xacro" />
@@ -39,8 +40,8 @@
     <link name="base_link"/>
     <!-- Build platform using robile bricks -->
-    <xacro:robile_active_wheel_brick name="robile_1" parent="base_link" movable_joints="$(arg movable_joints)">
+    <xacro:robile_active_wheel_brick name="robile_1" parent="base_link" movable_joints="$(arg movable_joints)" use_real_inertia="$(arg use_real_inertia)">
         <origin xyz="0.233 0.1165 0.05" rpy="0.0 0.0 0.0"/>
     </xacro:robile_active_wheel_brick>
-    <xacro:robile_active_wheel_brick name="robile_2" parent="base_link" movable_joints="$(arg movable_joints)">
+    <xacro:robile_active_wheel_brick name="robile_2" parent="base_link" movable_joints="$(arg movable_joints)" use_real_inertia="$(arg use_real_inertia)">
         <origin xyz="0.233 -0.1165 0.05" rpy="0.0 0.0 0.0"/>
     </xacro:robile_active_wheel_brick>
@@ -51,8 +52,8 @@
         <origin xyz="0.0 -0.1165 0.05" rpy="0.0 0.0 0.0"/>
     </xacro:robile_master_battery_brick>
-    <xacro:robile_active_wheel_brick name="robile_5" parent="base_link" movable_joints="$(arg movable_joints)">
+    <xacro:robile_active_wheel_brick name="robile_5" parent="base_link" movable_joints="$(arg movable_joints)" use_real_inertia="$(arg use_real_inertia)">
         <origin xyz="-0.233 0.1165 0.05" rpy="0.0 0.0 0.0"/>
     </xacro:robile_active_wheel_brick>
-    <xacro:robile_active_wheel_brick name="robile_6" parent="base_link" movable_joints="$(arg movable_joints)">
+    <xacro:robile_active_wheel_brick name="robile_6" parent="base_link" movable_joints="$(arg movable_joints)" use_real_inertia="$(arg use_real_inertia)">
         <origin xyz="-0.233 -0.1165 0.05" rpy="0.0 0.0 0.0"/>
     </xacro:robile_active_wheel_brick>

File: robots/6_wheel_config.urdf.xacro (robot description, xacro)
@@ -31,4 +31,5 @@
 <robot xmlns:xacro="http://ros.org/wiki/xacro" name="6_wheel_config" >
     <xacro:arg name="movable_joints" default="true"/>
+    <xacro:arg name="use_real_inertia" default="false"/>
     <!-- Include desired robile bricks -->
     <xacro:include filename="$(find robile_description)/urdf/robile_bricks/robile_active_wheel_brick.urdf.xacro" />
@@ -38,5 +39,5 @@
     <link name="base_link"/>
     <!-- Build platform using robile bricks -->
-    <xacro:robile_active_wheel_brick name="robile_1" parent="base_link" movable_joints="$(arg movable_joints)">
+    <xacro:robile_active_wheel_brick name="robile_1" parent="base_link" movable_joints="$(arg movable_joints)" use_real_inertia="$(arg use_real_inertia)">
         <origin xyz="0.233 0.466 0.05" rpy="0.0 0.0 0.0"/>
     </xacro:robile_active_wheel_brick>
@@ -44,5 +45,5 @@
         <origin xyz="0 0.466 0.05" rpy="0.0 0.0 0.0"/>
     </xacro:robile_empty_brick>
-    <xacro:robile_active_wheel_brick name="robile_3" parent="base_link" movable_joints="$(arg movable_joints)">
+    <xacro:robile_active_wheel_brick name="robile_3" parent="base_link" movable_joints="$(arg movable_joints)" use_real_inertia="$(arg use_real_inertia)">
         <origin xyz="-0.233 0.466 0.05" rpy="0.0 0.0 0.0"/>
     </xacro:robile_active_wheel_brick>
@@ -56,5 +57,5 @@
         <origin xyz="-0.233 0.233 0.05" rpy="0.0 0.0 0.0"/>
     </xacro:robile_empty_brick>
-    <xacro:robile_active_wheel_brick name="robile_7" parent="base_link" movable_joints="$(arg movable_joints)">
+    <xacro:robile_active_wheel_brick name="robile_7" parent="base_link" movable_joints="$(arg movable_joints)" use_real_inertia="$(arg use_real_inertia)">
         <origin xyz="0.233 0 0.05" rpy="0.0 0.0 0.0"/>
     </xacro:robile_active_wheel_brick>
@@ -62,5 +63,5 @@
         <origin xyz="0 0 0.05" rpy="0.0 0.0 0.0"/>
     </xacro:robile_empty_brick>
-    <xacro:robile_active_wheel_brick name="robile_9" parent="base_link" movable_joints="$(arg movable_joints)">
+    <xacro:robile_active_wheel_brick name="robile_9" parent="base_link" movable_joints="$(arg movable_joints)" use_real_inertia="$(arg use_real_inertia)">
         <origin xyz="-0.233 0 0.05" rpy="0.0 0.0 0.0"/>
     </xacro:robile_active_wheel_brick>
@@ -74,5 +75,5 @@
         <origin xyz="-0.233 -0.233 0.05" rpy="0.0 0.0 0.0"/>
     </xacro:robile_empty_brick>
-    <xacro:robile_active_wheel_brick name="robile_13" parent="base_link" movable_joints="$(arg movable_joints)">
+    <xacro:robile_active_wheel_brick name="robile_13" parent="base_link" movable_joints="$(arg movable_joints)" use_real_inertia="$(arg use_real_inertia)">
         <origin xyz="0.233 -0.466 0.05" rpy="0.0 0.0 0.0"/>
     </xacro:robile_active_wheel_brick>
@@ -80,5 +81,5 @@
         <origin xyz="0 -0.466 0.05" rpy="0.0 0.0 0.0"/>
     </xacro:robile_empty_brick>
-    <xacro:robile_active_wheel_brick name="robile_15" parent="base_link" movable_joints="$(arg movable_joints)">
+    <xacro:robile_active_wheel_brick name="robile_15" parent="base_link" movable_joints="$(arg movable_joints)" use_real_inertia="$(arg use_real_inertia)">
         <origin xyz="-0.233 -0.466 0.05" rpy="0.0 0.0 0.0"/>
     </xacro:robile_active_wheel_brick>

File: urdf/base_macros/kelo_drive.urdf.xacro (robot description, xacro)
@@ -30,5 +30,5 @@
 -->
 <robot xmlns:xacro="http://www.ros.org/wiki/xacro">
-    <xacro:macro name="kelo_drive" params="name parent *origin movable_joints:=true">
+    <xacro:macro name="kelo_drive" params="name parent *origin movable_joints:=true use_real_inertia:=false">
         <xacro:include filename="$(find robile_description)/urdf/base_macros/common.xacro" />
         <xacro:include filename="$(find robile_description)/urdf/base_macros/kelo_drive_wheel.urdf.xacro" />
@@ -108,9 +108,9 @@
         </joint>
         <!-- LEFT HUB WHEEL -->
-        <xacro:kelo_drive_wheel name="${name}_left_hub_wheel" parent="${name}_pivot_link" movable_joints="${movable_joints}">
+        <xacro:kelo_drive_wheel name="${name}_left_hub_wheel" parent="${name}_pivot_link" movable_joints="${movable_joints}" use_real_inertia="${use_real_inertia}">
             <origin xyz="-0.01 0.039326 0.001514" rpy="0 0 0.0"/>
         </xacro:kelo_drive_wheel>
         <!-- RIGHT HUB WHEEL -->
-        <xacro:kelo_drive_wheel name="${name}_right_hub_wheel" parent="${name}_pivot_link" movable_joints="${movable_joints}">
+        <xacro:kelo_drive_wheel name="${name}_right_hub_wheel" parent="${name}_pivot_link" movable_joints="${movable_joints}" use_real_inertia="${use_real_inertia}">
             <origin xyz="-0.01 -0.039326 0.001514" rpy="0 0 0.0"/>
         </xacro:kelo_drive_wheel>

File: urdf/base_macros/kelo_drive_wheel.urdf.xacro (robot description, xacro)
@@ -30,5 +30,5 @@
 -->
 <robot xmlns:xacro="http://www.ros.org/wiki/xacro">
-    <xacro:macro name="kelo_drive_wheel" params="name parent *origin movable_joints:=true">
+    <xacro:macro name="kelo_drive_wheel" params="name parent *origin movable_joints:=true use_real_inertia:=false">
         <xacro:include filename="$(find robile_description)/urdf/base_macros/common.xacro" />
         <xacro:if value="${movable_joints}">
@@ -71,9 +71,14 @@
                 </geometry>
             </collision>
-            <inertial>
-                <origin xyz="0 0 0" rpy="0 0 0"/>
-                <mass value="1.56317"/>
-                <inertia ixx="0.00101253363" ixy="0.00000000000" ixz="0.00000001020" iyy="0.00157998524" iyz="-0.00000055474" izz="0.00101282739"/>
-            </inertial>
+            <xacro:if value="${use_real_inertia}">
+                <inertial>
+                    <origin xyz="0 0 0" rpy="0 0 0"/>
+                    <mass value="1.56317"/>
+                    <inertia ixx="0.00101253363" ixy="0.00000000000" ixz="0.00000001020" iyy="0.00157998524" iyz="-0.00000055474" izz="0.00101282739"/>
+                </inertial>
+            </xacro:if>
+            <xacro:unless value="${use_real_inertia}">
+                <xacro:cuboid_inertia mass="10.0" length="0.233" breadth="0.233" height="0.233"/>
+            </xacro:unless>
         </link>
     </xacro:macro>

File: urdf/robile_bricks/robile_active_wheel_brick.urdf.xacro (robot description, xacro)
@@ -30,5 +30,5 @@
 -->
 <robot xmlns:xacro="http://www.ros.org/wiki/xacro">
-    <xacro:macro name="robile_active_wheel_brick" params="name parent *origin movable_joints:=true">
+    <xacro:macro name="robile_active_wheel_brick" params="name parent *origin movable_joints:=true use_real_inertia:=false">
         <!-- Include xacro files-->
         <xacro:include filename="$(find robile_description)/urdf/base_macros/brick_housing.urdf.xacro" />
@@ -40,5 +40,5 @@
         </joint>
         <xacro:brick_housing name="${name}" with_wheel="true" color="red"/>
-        <xacro:kelo_drive name="${name}_drive" parent="${name}_link" movable_joints="${movable_joints}">
+        <xacro:kelo_drive name="${name}_drive" parent="${name}_link" movable_joints="${movable_joints}" use_real_inertia="${use_real_inertia}">
             <origin xyz="0 0 0" rpy="0 0 0.0"/>
         </xacro:kelo_drive>
