Commit message: Remove movable_joints argument from xacro files

File: robots/2_wheel_config.urdf.xacro (robot description, xacro)
@@ -30,5 +30,4 @@
 -->
 <robot xmlns:xacro="http://ros.org/wiki/xacro" name="2_wheel_config" >
-    <xacro:arg name="movable_joints" default="true"/>
     <xacro:arg name="use_real_inertia" default="false"/>
     <!-- Include desired robile bricks -->
@@ -39,8 +38,8 @@
     <link name="base_link"/>
     <!-- Build platform using robile bricks -->
-    <xacro:robile_passive_wheel_brick name="robile_1" parent="base_link" movable_joints="$(arg movable_joints)">
+    <xacro:robile_passive_wheel_brick name="robile_1" parent="base_link">
         <origin xyz="0.233 0.1165 0.05" rpy="0.0 0.0 0.0"/>
     </xacro:robile_passive_wheel_brick>
-    <xacro:robile_passive_wheel_brick name="robile_2" parent="base_link" movable_joints="$(arg movable_joints)">
+    <xacro:robile_passive_wheel_brick name="robile_2" parent="base_link">
         <origin xyz="0.233 -0.1165 0.05" rpy="0.0 0.0 0.0"/>
     </xacro:robile_passive_wheel_brick>
@@ -51,8 +50,8 @@
         <origin xyz="0.0 -0.1165 0.05" rpy="0.0 0.0 0.0"/>
     </xacro:robile_master_battery_brick>
-    <xacro:robile_active_wheel_brick name="robile_5" parent="base_link" movable_joints="$(arg movable_joints)" use_real_inertia="$(arg use_real_inertia)">
+    <xacro:robile_active_wheel_brick name="robile_5" parent="base_link" use_real_inertia="$(arg use_real_inertia)">
         <origin xyz="-0.233 0.1165 0.05" rpy="0.0 0.0 0.0"/>
     </xacro:robile_active_wheel_brick>
-    <xacro:robile_active_wheel_brick name="robile_6" parent="base_link" movable_joints="$(arg movable_joints)" use_real_inertia="$(arg use_real_inertia)">
+    <xacro:robile_active_wheel_brick name="robile_6" parent="base_link" use_real_inertia="$(arg use_real_inertia)">
         <origin xyz="-0.233 -0.1165 0.05" rpy="0.0 0.0 0.0"/>
     </xacro:robile_active_wheel_brick>

File: robots/4_wheel_config.urdf.xacro (robot description, xacro)
@@ -30,5 +30,4 @@
 -->
 <robot xmlns:xacro="http://ros.org/wiki/xacro" name="4_wheel_config" >
-    <xacro:arg name="movable_joints" default="true"/>
     <xacro:arg name="use_real_inertia" default="false"/>
     <!-- Include desired robile bricks -->
@@ -38,8 +37,8 @@
     <link name="base_link"/>
     <!-- Build platform using robile bricks -->
-    <xacro:robile_active_wheel_brick name="robile_1" parent="base_link" movable_joints="$(arg movable_joints)" use_real_inertia="$(arg use_real_inertia)">
+    <xacro:robile_active_wheel_brick name="robile_1" parent="base_link" use_real_inertia="$(arg use_real_inertia)">
         <origin xyz="0.233 0.1165 0.05" rpy="0.0 0.0 0.0"/>
     </xacro:robile_active_wheel_brick>
-    <xacro:robile_active_wheel_brick name="robile_2" parent="base_link" movable_joints="$(arg movable_joints)" use_real_inertia="$(arg use_real_inertia)">
+    <xacro:robile_active_wheel_brick name="robile_2" parent="base_link" use_real_inertia="$(arg use_real_inertia)">
         <origin xyz="0.233 -0.1165 0.05" rpy="0.0 0.0 0.0"/>
     </xacro:robile_active_wheel_brick>
@@ -50,8 +49,8 @@
         <origin xyz="0.0 -0.1165 0.05" rpy="0.0 0.0 0.0"/>
     </xacro:robile_master_battery_brick>
-    <xacro:robile_active_wheel_brick name="robile_5" parent="base_link" movable_joints="$(arg movable_joints)" use_real_inertia="$(arg use_real_inertia)">
+    <xacro:robile_active_wheel_brick name="robile_5" parent="base_link" use_real_inertia="$(arg use_real_inertia)">
         <origin xyz="-0.233 0.1165 0.05" rpy="0.0 0.0 0.0"/>
     </xacro:robile_active_wheel_brick>
-    <xacro:robile_active_wheel_brick name="robile_6" parent="base_link" movable_joints="$(arg movable_joints)" use_real_inertia="$(arg use_real_inertia)">
+    <xacro:robile_active_wheel_brick name="robile_6" parent="base_link" use_real_inertia="$(arg use_real_inertia)">
         <origin xyz="-0.233 -0.1165 0.05" rpy="0.0 0.0 0.0"/>
     </xacro:robile_active_wheel_brick>

File: robots/4_wheel_double_microscan_config.urdf.xacro (robot description, xacro)
@@ -31,5 +31,4 @@
 -->
 <robot xmlns:xacro="http://ros.org/wiki/xacro" name="4_wheel_double_microscan_config" >
-    <xacro:arg name="movable_joints" default="true"/>
     <xacro:arg name="use_real_inertia" default="false"/>
     <!-- Include desired robile bricks -->
@@ -40,8 +39,8 @@
     <link name="base_link"/>
     <!-- Build platform using robile bricks -->
-    <xacro:robile_active_wheel_brick name="robile_1" parent="base_link" movable_joints="$(arg movable_joints)" use_real_inertia="$(arg use_real_inertia)">
+    <xacro:robile_active_wheel_brick name="robile_1" parent="base_link" use_real_inertia="$(arg use_real_inertia)">
         <origin xyz="0.233 0.1165 0.05" rpy="0.0 0.0 0.0"/>
     </xacro:robile_active_wheel_brick>
-    <xacro:robile_active_wheel_brick name="robile_2" parent="base_link" movable_joints="$(arg movable_joints)" use_real_inertia="$(arg use_real_inertia)">
+    <xacro:robile_active_wheel_brick name="robile_2" parent="base_link" use_real_inertia="$(arg use_real_inertia)">
         <origin xyz="0.233 -0.1165 0.05" rpy="0.0 0.0 0.0"/>
     </xacro:robile_active_wheel_brick>
@@ -52,8 +51,8 @@
         <origin xyz="0.0 -0.1165 0.05" rpy="0.0 0.0 0.0"/>
     </xacro:robile_master_battery_brick>
-    <xacro:robile_active_wheel_brick name="robile_5" parent="base_link" movable_joints="$(arg movable_joints)" use_real_inertia="$(arg use_real_inertia)">
+    <xacro:robile_active_wheel_brick name="robile_5" parent="base_link" use_real_inertia="$(arg use_real_inertia)">
         <origin xyz="-0.233 0.1165 0.05" rpy="0.0 0.0 0.0"/>
     </xacro:robile_active_wheel_brick>
-    <xacro:robile_active_wheel_brick name="robile_6" parent="base_link" movable_joints="$(arg movable_joints)" use_real_inertia="$(arg use_real_inertia)">
+    <xacro:robile_active_wheel_brick name="robile_6" parent="base_link" use_real_inertia="$(arg use_real_inertia)">
         <origin xyz="-0.233 -0.1165 0.05" rpy="0.0 0.0 0.0"/>
     </xacro:robile_active_wheel_brick>

File: robots/4_wheel_double_uam_config.urdf.xacro (robot description, xacro)
@@ -31,5 +31,4 @@
 -->
 <robot xmlns:xacro="http://ros.org/wiki/xacro" name="4_wheel_double_microscan_config" >
-    <xacro:arg name="movable_joints" default="true"/>
     <xacro:arg name="use_real_inertia" default="false"/>
     <!-- Include desired robile bricks -->
@@ -40,8 +39,8 @@
     <link name="base_link"/>
     <!-- Build platform using robile bricks -->
-    <xacro:robile_active_wheel_brick name="robile_1" parent="base_link" movable_joints="$(arg movable_joints)" use_real_inertia="$(arg use_real_inertia)">
+    <xacro:robile_active_wheel_brick name="robile_1" parent="base_link" use_real_inertia="$(arg use_real_inertia)">
         <origin xyz="0.233 0.1165 0.05" rpy="0.0 0.0 0.0"/>
     </xacro:robile_active_wheel_brick>
-    <xacro:robile_active_wheel_brick name="robile_2" parent="base_link" movable_joints="$(arg movable_joints)" use_real_inertia="$(arg use_real_inertia)">
+    <xacro:robile_active_wheel_brick name="robile_2" parent="base_link" use_real_inertia="$(arg use_real_inertia)">
         <origin xyz="0.233 -0.1165 0.05" rpy="0.0 0.0 0.0"/>
     </xacro:robile_active_wheel_brick>
@@ -52,8 +51,8 @@
         <origin xyz="0.0 -0.1165 0.05" rpy="0.0 0.0 0.0"/>
     </xacro:robile_master_battery_brick>
-    <xacro:robile_active_wheel_brick name="robile_5" parent="base_link" movable_joints="$(arg movable_joints)" use_real_inertia="$(arg use_real_inertia)">
+    <xacro:robile_active_wheel_brick name="robile_5" parent="base_link" use_real_inertia="$(arg use_real_inertia)">
         <origin xyz="-0.233 0.1165 0.05" rpy="0.0 0.0 0.0"/>
     </xacro:robile_active_wheel_brick>
-    <xacro:robile_active_wheel_brick name="robile_6" parent="base_link" movable_joints="$(arg movable_joints)" use_real_inertia="$(arg use_real_inertia)">
+    <xacro:robile_active_wheel_brick name="robile_6" parent="base_link" use_real_inertia="$(arg use_real_inertia)">
         <origin xyz="-0.233 -0.1165 0.05" rpy="0.0 0.0 0.0"/>
     </xacro:robile_active_wheel_brick>

File: robots/4_wheel_lidar_config.urdf.xacro (robot description, xacro)
@@ -31,5 +31,4 @@
 -->
 <robot xmlns:xacro="http://ros.org/wiki/xacro" name="4_wheel_lidar_config" >
-    <xacro:arg name="movable_joints" default="true"/>
     <xacro:arg name="use_real_inertia" default="false"/>
     <!-- Include desired robile bricks -->
@@ -40,8 +39,8 @@
     <link name="base_link"/>
     <!-- Build platform using robile bricks -->
-    <xacro:robile_active_wheel_brick name="robile_1" parent="base_link" movable_joints="$(arg movable_joints)" use_real_inertia="$(arg use_real_inertia)">
+    <xacro:robile_active_wheel_brick name="robile_1" parent="base_link" use_real_inertia="$(arg use_real_inertia)">
         <origin xyz="0.233 0.1165 0.05" rpy="0.0 0.0 0.0"/>
     </xacro:robile_active_wheel_brick>
-    <xacro:robile_active_wheel_brick name="robile_2" parent="base_link" movable_joints="$(arg movable_joints)" use_real_inertia="$(arg use_real_inertia)">
+    <xacro:robile_active_wheel_brick name="robile_2" parent="base_link" use_real_inertia="$(arg use_real_inertia)">
         <origin xyz="0.233 -0.1165 0.05" rpy="0.0 0.0 0.0"/>
     </xacro:robile_active_wheel_brick>
@@ -52,8 +51,8 @@
         <origin xyz="0.0 -0.1165 0.05" rpy="0.0 0.0 0.0"/>
     </xacro:robile_master_battery_brick>
-    <xacro:robile_active_wheel_brick name="robile_5" parent="base_link" movable_joints="$(arg movable_joints)" use_real_inertia="$(arg use_real_inertia)">
+    <xacro:robile_active_wheel_brick name="robile_5" parent="base_link" use_real_inertia="$(arg use_real_inertia)">
         <origin xyz="-0.233 0.1165 0.05" rpy="0.0 0.0 0.0"/>
     </xacro:robile_active_wheel_brick>
-    <xacro:robile_active_wheel_brick name="robile_6" parent="base_link" movable_joints="$(arg movable_joints)" use_real_inertia="$(arg use_real_inertia)">
+    <xacro:robile_active_wheel_brick name="robile_6" parent="base_link" use_real_inertia="$(arg use_real_inertia)">
         <origin xyz="-0.233 -0.1165 0.05" rpy="0.0 0.0 0.0"/>
     </xacro:robile_active_wheel_brick>

File: robots/6_wheel_config.urdf.xacro (robot description, xacro)
@@ -30,5 +30,4 @@
 -->
 <robot xmlns:xacro="http://ros.org/wiki/xacro" name="6_wheel_config" >
-    <xacro:arg name="movable_joints" default="true"/>
     <xacro:arg name="use_real_inertia" default="false"/>
     <!-- Include desired robile bricks -->
@@ -39,5 +38,5 @@
     <link name="base_link"/>
     <!-- Build platform using robile bricks -->
-    <xacro:robile_active_wheel_brick name="robile_1" parent="base_link" movable_joints="$(arg movable_joints)" use_real_inertia="$(arg use_real_inertia)">
+    <xacro:robile_active_wheel_brick name="robile_1" parent="base_link" use_real_inertia="$(arg use_real_inertia)">
         <origin xyz="0.233 0.466 0.05" rpy="0.0 0.0 0.0"/>
     </xacro:robile_active_wheel_brick>
@@ -45,5 +44,5 @@
         <origin xyz="0 0.466 0.05" rpy="0.0 0.0 0.0"/>
     </xacro:robile_empty_brick>
-    <xacro:robile_active_wheel_brick name="robile_3" parent="base_link" movable_joints="$(arg movable_joints)" use_real_inertia="$(arg use_real_inertia)">
+    <xacro:robile_active_wheel_brick name="robile_3" parent="base_link" use_real_inertia="$(arg use_real_inertia)">
         <origin xyz="-0.233 0.466 0.05" rpy="0.0 0.0 0.0"/>
     </xacro:robile_active_wheel_brick>
@@ -57,5 +56,5 @@
         <origin xyz="-0.233 0.233 0.05" rpy="0.0 0.0 0.0"/>
     </xacro:robile_empty_brick>
-    <xacro:robile_active_wheel_brick name="robile_7" parent="base_link" movable_joints="$(arg movable_joints)" use_real_inertia="$(arg use_real_inertia)">
+    <xacro:robile_active_wheel_brick name="robile_7" parent="base_link" use_real_inertia="$(arg use_real_inertia)">
         <origin xyz="0.233 0 0.05" rpy="0.0 0.0 0.0"/>
     </xacro:robile_active_wheel_brick>
@@ -63,5 +62,5 @@
         <origin xyz="0 0 0.05" rpy="0.0 0.0 0.0"/>
     </xacro:robile_empty_brick>
-    <xacro:robile_active_wheel_brick name="robile_9" parent="base_link" movable_joints="$(arg movable_joints)" use_real_inertia="$(arg use_real_inertia)">
+    <xacro:robile_active_wheel_brick name="robile_9" parent="base_link" use_real_inertia="$(arg use_real_inertia)">
         <origin xyz="-0.233 0 0.05" rpy="0.0 0.0 0.0"/>
     </xacro:robile_active_wheel_brick>
@@ -75,5 +74,5 @@
         <origin xyz="-0.233 -0.233 0.05" rpy="0.0 0.0 0.0"/>
     </xacro:robile_empty_brick>
-    <xacro:robile_active_wheel_brick name="robile_13" parent="base_link" movable_joints="$(arg movable_joints)" use_real_inertia="$(arg use_real_inertia)">
+    <xacro:robile_active_wheel_brick name="robile_13" parent="base_link" use_real_inertia="$(arg use_real_inertia)">
         <origin xyz="0.233 -0.466 0.05" rpy="0.0 0.0 0.0"/>
     </xacro:robile_active_wheel_brick>
@@ -81,5 +80,5 @@
         <origin xyz="0 -0.466 0.05" rpy="0.0 0.0 0.0"/>
     </xacro:robile_empty_brick>
-    <xacro:robile_active_wheel_brick name="robile_15" parent="base_link" movable_joints="$(arg movable_joints)" use_real_inertia="$(arg use_real_inertia)">
+    <xacro:robile_active_wheel_brick name="robile_15" parent="base_link" use_real_inertia="$(arg use_real_inertia)">
         <origin xyz="-0.233 -0.466 0.05" rpy="0.0 0.0 0.0"/>
     </xacro:robile_active_wheel_brick>

File: urdf/base_macros/kelo_drive.urdf.xacro (robot description, xacro)
@@ -30,34 +30,23 @@
 -->
 <robot xmlns:xacro="http://www.ros.org/wiki/xacro">
-    <xacro:macro name="kelo_drive" params="name parent *origin movable_joints:=true use_real_inertia:=false">
+    <xacro:macro name="kelo_drive" params="name parent *origin use_real_inertia:=false">
         <xacro:include filename="$(find robile_description)/urdf/base_macros/common.xacro" />
         <xacro:include filename="$(find robile_description)/urdf/base_macros/kelo_drive_wheel.urdf.xacro" />
-        <!-- PIVOT -->
-        <xacro:if value="${movable_joints}">
-            <joint name="${name}_pivot_joint" type="continuous">
-                <xacro:insert_block name="origin" />
-                <axis xyz="0 0 1"/>
-                <parent link="${parent}"/>
-                <child link="${name}_pivot_link" />
+        <joint name="${name}_pivot_joint" type="continuous">
+            <xacro:insert_block name="origin" />
+            <axis xyz="0 0 1"/>
+            <parent link="${parent}"/>
+            <child link="${name}_pivot_link" />
+        </joint>
+        <transmission name="${name}_pivot_transmission">
+            <type>transmission_interface/SimpleTransmission</type>
+            <joint name="${name}_pivot_joint">
+                <hardwareInterface>hardware_interface/EffortJointInterface</hardwareInterface>
             </joint>
-            <transmission name="${name}_pivot_transmission">
-                <type>transmission_interface/SimpleTransmission</type>
-                <joint name="${name}_pivot_joint">
-                    <hardwareInterface>hardware_interface/EffortJointInterface</hardwareInterface>
-                </joint>
-                <actuator name="${name}_pivot_motor">
-                    <hardwareInterface>hardware_interface/EffortJointInterface</hardwareInterface>
-                    <mechanicalReduction>1</mechanicalReduction>
-                </actuator>
-            </transmission>
-        </xacro:if>
-        <xacro:unless value="${movable_joints}">
-            <joint name="${name}_pivot_joint" type="fixed">
-                <xacro:insert_block name="origin" />
-                <axis xyz="0 0 1"/>
-                <parent link="${parent}"/>
-                <child link="${name}_pivot_link" />
-            </joint>
-        </xacro:unless>
+            <actuator name="${name}_pivot_motor">
+                <hardwareInterface>hardware_interface/EffortJointInterface</hardwareInterface>
+                <mechanicalReduction>1</mechanicalReduction>
+            </actuator>
+        </transmission>
         <link name="${name}_pivot_link">
             <visual>
@@ -108,9 +97,9 @@
         </joint>
         <!-- LEFT HUB WHEEL -->
-        <xacro:kelo_drive_wheel name="${name}_left_hub_wheel" parent="${name}_pivot_link" movable_joints="${movable_joints}" use_real_inertia="${use_real_inertia}">
+        <xacro:kelo_drive_wheel name="${name}_left_hub_wheel" parent="${name}_pivot_link" use_real_inertia="${use_real_inertia}">
             <origin xyz="-0.01 0.039326 0.001514" rpy="0 0 0.0"/>
         </xacro:kelo_drive_wheel>
         <!-- RIGHT HUB WHEEL -->
-        <xacro:kelo_drive_wheel name="${name}_right_hub_wheel" parent="${name}_pivot_link" movable_joints="${movable_joints}" use_real_inertia="${use_real_inertia}">
+        <xacro:kelo_drive_wheel name="${name}_right_hub_wheel" parent="${name}_pivot_link" use_real_inertia="${use_real_inertia}">
             <origin xyz="-0.01 -0.039326 0.001514" rpy="0 0 0.0"/>
         </xacro:kelo_drive_wheel>

File: urdf/base_macros/kelo_drive_wheel.urdf.xacro (robot description, xacro)
@@ -30,32 +30,22 @@
 -->
 <robot xmlns:xacro="http://www.ros.org/wiki/xacro">
-    <xacro:macro name="kelo_drive_wheel" params="name parent *origin movable_joints:=true use_real_inertia:=false">
+    <xacro:macro name="kelo_drive_wheel" params="name parent *origin use_real_inertia:=false">
         <xacro:include filename="$(find robile_description)/urdf/base_macros/common.xacro" />
-        <xacro:if value="${movable_joints}">
-            <joint name="${name}_joint" type="continuous">
-                <xacro:insert_block name="origin" />
-                <axis xyz="0 1 0"/>
-                <parent link="${parent}"/>
-                <child link="${name}_link" />
+        <joint name="${name}_joint" type="continuous">
+            <xacro:insert_block name="origin" />
+            <axis xyz="0 1 0"/>
+            <parent link="${parent}"/>
+            <child link="${name}_link" />
+        </joint>
+        <transmission name="${name}_transmission">
+            <type>transmission_interface/SimpleTransmission</type>
+            <joint name="${name}_joint">
+                <hardwareInterface>hardware_interface/EffortJointInterface</hardwareInterface>
             </joint>
-            <transmission name="${name}_transmission">
-                <type>transmission_interface/SimpleTransmission</type>
-                <joint name="${name}_joint">
-                    <hardwareInterface>hardware_interface/EffortJointInterface</hardwareInterface>
-                </joint>
-                <actuator name="${name}_motor">
-                    <hardwareInterface>hardware_interface/EffortJointInterface</hardwareInterface>
-                    <mechanicalReduction>1</mechanicalReduction>
-                </actuator>
-            </transmission>
-        </xacro:if>
-        <xacro:unless value="${movable_joints}">
-            <joint name="${name}_joint" type="fixed">
-                <xacro:insert_block name="origin" />
-                <axis xyz="0 1 0"/>
-                <parent link="${parent}"/>
-                <child link="${name}_link" />
-            </joint>
-        </xacro:unless>
+            <actuator name="${name}_motor">
+                <hardwareInterface>hardware_interface/EffortJointInterface</hardwareInterface>
+                <mechanicalReduction>1</mechanicalReduction>
+            </actuator>
+        </transmission>
         <link name="${name}_link">
             <visual>
