Commit message: Remove movable_joints argument from xacro files

File: urdf/base_macros/passive_caster_wheel.urdf.xacro (robot description, xacro)
@@ -30,33 +30,22 @@
 -->
 <robot xmlns:xacro="http://www.ros.org/wiki/xacro">
-    <xacro:macro name="passive_caster_wheel" params="name parent *origin movable_joints:=true">
+    <xacro:macro name="passive_caster_wheel" params="name parent *origin">
         <xacro:include filename="$(find robile_description)/urdf/base_macros/common.xacro" />
-        <!-- PIVOT -->
-        <xacro:if value="${movable_joints}">
-            <joint name="${name}_pivot_caster_joint" type="continuous">
-                <xacro:insert_block name="origin" />
-                <axis xyz="0 0 1"/>
-                <parent link="${parent}"/>
-                <child link="${name}_pivot_link" />
+        <joint name="${name}_pivot_caster_joint" type="continuous">
+            <xacro:insert_block name="origin" />
+            <axis xyz="0 0 1"/>
+            <parent link="${parent}"/>
+            <child link="${name}_pivot_link" />
+        </joint>
+        <transmission name="${name}_pivot_transmission">
+            <type>transmission_interface/SimpleTransmission</type>
+            <joint name="${name}_pivot_caster_joint">
+                <hardwareInterface>hardware_interface/EffortJointInterface</hardwareInterface>
             </joint>
-            <transmission name="${name}_pivot_transmission">
-                <type>transmission_interface/SimpleTransmission</type>
-                <joint name="${name}_pivot_caster_joint">
-                    <hardwareInterface>hardware_interface/EffortJointInterface</hardwareInterface>
-                </joint>
-                <actuator name="${name}_pivot_motor">
-                    <hardwareInterface>hardware_interface/EffortJointInterface</hardwareInterface>
-                    <mechanicalReduction>1</mechanicalReduction>
-                </actuator>
-            </transmission>
-        </xacro:if>
-        <xacro:unless value="${movable_joints}">
-            <joint name="${name}_pivot_caster_joint" type="fixed">
-                <xacro:insert_block name="origin" />
-                <axis xyz="0 0 1"/>
-                <parent link="${parent}"/>
-                <child link="${name}_pivot_link" />
-            </joint>
-        </xacro:unless>
+            <actuator name="${name}_pivot_motor">
+                <hardwareInterface>hardware_interface/EffortJointInterface</hardwareInterface>
+                <mechanicalReduction>1</mechanicalReduction>
+            </actuator>
+        </transmission>
         <link name="${name}_pivot_link">
             <visual>
@@ -78,30 +67,20 @@
         </link>
         <!-- CASTER WHEEL -->
-        <xacro:if value="${movable_joints}">
-            <joint name="${name}_wheel_joint" type="continuous">
-                <origin xyz="0 0 0" rpy="0 0 0"/>
-                <axis xyz="0 1 0"/>
-                <parent link="${name}_caster_offset_link"/>
-                <child link="${name}_wheel_link" />
+        <joint name="${name}_wheel_joint" type="continuous">
+            <origin xyz="0 0 0" rpy="0 0 0"/>
+            <axis xyz="0 1 0"/>
+            <parent link="${name}_caster_offset_link"/>
+            <child link="${name}_wheel_link" />
+        </joint>
+        <transmission name="${name}_wheel_transmission">
+            <type>transmission_interface/SimpleTransmission</type>
+            <joint name="${name}_wheel_joint">
+                <hardwareInterface>hardware_interface/EffortJointInterface</hardwareInterface>
             </joint>
-            <transmission name="${name}_wheel_transmission">
-                <type>transmission_interface/SimpleTransmission</type>
-                <joint name="${name}_wheel_joint">
-                    <hardwareInterface>hardware_interface/EffortJointInterface</hardwareInterface>
-                </joint>
-                <actuator name="${name}_wheel_motor">
-                    <hardwareInterface>hardware_interface/EffortJointInterface</hardwareInterface>
-                    <mechanicalReduction>1</mechanicalReduction>
-                </actuator>
-            </transmission>
-        </xacro:if>
-        <xacro:unless value="${movable_joints}">
-            <joint name="${name}_wheel_joint" type="fixed">
-                <origin xyz="0 0 0" rpy="0 0 0"/>
-                <axis xyz="0 1 0"/>
-                <parent link="${name}_caster_offset_link"/>
-                <child link="${name}_wheel_link" />
-            </joint>
-        </xacro:unless>
+            <actuator name="${name}_wheel_motor">
+                <hardwareInterface>hardware_interface/EffortJointInterface</hardwareInterface>
+                <mechanicalReduction>1</mechanicalReduction>
+            </actuator>
+        </transmission>
         <link name="${name}_wheel_link">
             <visual>

File: urdf/robile_bricks/robile_active_wheel_brick.urdf.xacro (robot description, xacro)
@@ -30,5 +30,5 @@
 -->
 <robot xmlns:xacro="http://www.ros.org/wiki/xacro">
-    <xacro:macro name="robile_active_wheel_brick" params="name parent *origin movable_joints:=true use_real_inertia:=false">
+    <xacro:macro name="robile_active_wheel_brick" params="name parent *origin use_real_inertia:=false">
         <!-- Include xacro files-->
         <xacro:include filename="$(find robile_description)/urdf/base_macros/brick_housing.urdf.xacro" />
@@ -40,5 +40,5 @@
         </joint>
         <xacro:brick_housing name="${name}" with_wheel="true" color="red"/>
-        <xacro:kelo_drive name="${name}_drive" parent="${name}_link" movable_joints="${movable_joints}" use_real_inertia="${use_real_inertia}">
+        <xacro:kelo_drive name="${name}_drive" parent="${name}_link" use_real_inertia="${use_real_inertia}">
             <origin xyz="0 0 0" rpy="0 0 0.0"/>
         </xacro:kelo_drive>

File: urdf/robile_bricks/robile_passive_wheel_brick.urdf.xacro (robot description, xacro)
@@ -30,5 +30,5 @@
 -->
 <robot xmlns:xacro="http://www.ros.org/wiki/xacro">
-    <xacro:macro name="robile_passive_wheel_brick" params="name parent *origin movable_joints:=true">
+    <xacro:macro name="robile_passive_wheel_brick" params="name parent *origin">
         <!-- Include xacro files-->
         <xacro:include filename="$(find robile_description)/urdf/base_macros/brick_housing.urdf.xacro" />
@@ -40,5 +40,5 @@
         </joint>
         <xacro:brick_housing name="${name}" with_wheel="true" color="blue"/>
-        <xacro:passive_caster_wheel name="${name}_caster_wheel" parent="${name}_link" movable_joints="${movable_joints}">
+        <xacro:passive_caster_wheel name="${name}_caster_wheel" parent="${name}_link">
             <origin xyz="0 0 0" rpy="0 0 0.0"/>
         </xacro:passive_caster_wheel>
