Commit message: Update sensor plugins for ROS2 Gazebo Ignition

File: urdf/sensors/common.xacro (robot description, xacro)
@@ -1,43 +1,36 @@
 <?xml version="1.0"?>
 <robot xmlns:xacro="http://www.ros.org/wiki/xacro">
-    <xacro:macro name="gazebo_laser_plugin" params="name topic sample_size
-                                                    update_rate min_angle
-                                                    max_angle min_range max_range
-                                                    robot_namespace visualize
-                                                    sensor_type:=gpu_ray
-                                                    plugin_filename:=libgazebo_ros_gpu_laser" >
-        <gazebo reference="${name}_link">
-            <!-- <turnGravityOff>true</turnGravityOff> -->
-            <sensor type="${sensor_type}" name="${name}">
-                <pose>0 0 0 0 0 0</pose>
-                <visualize>${visualize}</visualize>
-                <update_rate>${update_rate}</update_rate>
-                <ray>
-                    <scan>
-                        <horizontal>
-                            <samples>${sample_size}</samples>
-                            <resolution>1</resolution>
-                            <min_angle>${min_angle}</min_angle>
-                            <max_angle>${max_angle}</max_angle>
-                        </horizontal>
-                    </scan>
-                    <range>
-                        <min>${min_range}</min>
-                        <max>${max_range}</max>
-                        <resolution>0.01</resolution>
-                    </range>
-                    <noise>
-                        <type>gaussian</type>
-                        <mean>0.0</mean>
-                        <stddev>0.005</stddev>
-                    </noise>
-                </ray>
-                <plugin name="${name}_controller" filename="${plugin_filename}.so">
-                    <topicName>${topic}</topicName>
-                    <frameName>${name}_link</frameName>
-                    <robotNamespace>${robot_namespace}</robotNamespace>
-                </plugin>
-            </sensor>
-        </gazebo>
+    <xacro:macro name="gazebo_laser_plugin" params="name topic sample_size update_rate
+                                                    min_angle max_angle min_range max_range
+                                                    visualize sensor_type:=gpu_lidar " >
+    <gazebo reference="${name}_link">
+        <sensor type="${sensor_type}" name="${name}">
+            <pose>0 0 0 0 0 0</pose>
+            <visualize>${visualize}</visualize>
+            <update_rate>${update_rate}</update_rate>
+            <lidar>
+                <scan>
+                    <horizontal>
+                        <samples>${sample_size}</samples>
+                        <resolution>1</resolution>
+                        <min_angle>${min_angle}</min_angle>
+                        <max_angle>${max_angle}</max_angle>
+                    </horizontal>
+                </scan>
+                <range>
+                    <min>${min_range}</min>
+                    <max>${max_range}</max>
+                    <resolution>0.01</resolution>
+                </range>
+                <noise>
+                    <type>gaussian</type>
+                    <mean>0.0</mean>
+                    <stddev>0.005</stddev>
+                </noise>
+            </lidar>
+            <topic>${topic}</topic>
+            <gz_frame_id>${name}_link</gz_frame_id>
+        </sensor>
+    </gazebo>
     </xacro:macro>
 </robot>

File: urdf/sensors/datalogic.urdf.xacro (robot description, xacro)
@@ -32,7 +32,5 @@
                                           sample_size:=540 update_rate:=10
                                           min_angle:=-2.35619 max_angle:=2.35619
-                                          min_range:=0.1 max_range:=30.0
-                                          robot_namespace:=/ use_gpu:=true
-                                          visualize:=false" >
+                                          min_range:=0.1 max_range:=30.0 visualize:=true">
         <joint name="${name}_joint" type="fixed">
             <axis xyz="0 1 0" />
@@ -63,18 +61,7 @@
             </collision>
         </link>
-        <xacro:if value="${use_gpu}">
-            <xacro:gazebo_laser_plugin name="${name}" topic="${topic}" sample_size="${sample_size}"
-                                       update_rate="${update_rate}" min_angle="${min_angle}"
-                                       max_angle="${max_angle}" min_range="${min_range}" max_range="${max_range}"
-                                       robot_namespace="${robot_namespace}" visualize="${visualize}"
-                                       sensor_type="gpu_ray" plugin_filename="libgazebo_ros_gpu_laser"/>
-        </xacro:if>
-        <xacro:unless value="${use_gpu}">
-            <xacro:gazebo_laser_plugin name="${name}" topic="${topic}" sample_size="${sample_size}"
-                                       update_rate="${update_rate}" min_angle="${min_angle}"
-                                       max_angle="${max_angle}" min_range="${min_range}" max_range="${max_range}"
-                                       robot_namespace="${robot_namespace}" visualize="${visualize}"
-                                       sensor_type="ray" plugin_filename="libgazebo_ros_laser"/>
-        </xacro:unless>
+        <xacro:gazebo_laser_plugin name="${name}" topic="${topic}" sample_size="${sample_size}" update_rate="${update_rate}"
+                                min_angle="${min_angle}" max_angle="${max_angle}" min_range="${min_range}" max_range="${max_range}"
+                                visualize="${visualize}" sensor_type="gpu_lidar"/>
     </xacro:macro>
 </robot>

File: urdf/sensors/hokuyo_uam_05lpa.urdf.xacro (robot description, xacro)
@@ -1,30 +1,38 @@
 <?xml version="1.0"?>
-<robot xmlns:xacro="http://www.ros.org/wiki/xacro" name="kelo">
-  <xacro:macro name="hokuyo_uam_05lpa" params="name parent *origin ros_topic">
-    <joint name="${name}_joint" type="fixed">
-      <axis xyz="0 1 0" />
-      <xacro:insert_block name="origin" />
-      <parent link="${parent}"/>
-      <child link="${name}_link"/>
-    </joint>
-    <link name="${name}_link" type="laser">
-      <inertial>
-        <mass value="0.001" />
-        <origin xyz="0 0 0" rpy="0 0 0" />
-        <inertia ixx="0.0001" ixy="0" ixz="0" iyy="0.000001" iyz="0" izz="0.0001" />
-      </inertial>
-      <visual>
-        <origin xyz="0 0 0" rpy="1.57 0 1.57" />
-      <geometry>
-        <mesh filename="package://robile_description/meshes/sensors/UAM-05LPA.dae" scale="1 1 1" />
-        </geometry>
-      </visual>
-      <collision>
-        <origin xyz="0 0 0" rpy="1.57 0 1.57" />
-        <geometry>
-          <mesh filename="package://robile_description/meshes/sensors/UAM-05LPA.dae" scale="1 1 1" />
-        </geometry>
-      </collision>
-    </link>
+<robot xmlns:xacro="http://www.ros.org/wiki/xacro">
+  <xacro:include filename="$(find robile_description)/urdf/sensors/common.xacro" />
+  <xacro:macro name="hokuyo_uam_05lpa" params="*origin name:=base_laser_front
+                                          ros_topic parent:=base_link
+                                          sample_size:=540 update_rate:=10
+                                          min_angle:=-2.35619 max_angle:=2.35619
+                                          min_range:=0.1 max_range:=40.0 visualize:=true">
+      <joint name="${name}_joint" type="fixed">
+          <axis xyz="0 1 0" />
+          <xacro:insert_block name="origin" />
+          <parent link="${parent}" />
+          <child link="${name}_link" />
+      </joint>
+      <link name="${name}_link" type="laser">
+          <inertial>
+              <mass value="0.001" />
+              <origin xyz="0 0 0" rpy="0 0 0" />
+              <inertia ixx="0.0001" ixy="0" ixz="0" iyy="0.000001" iyz="0" izz="0.0001" />
+          </inertial>
+          <visual>
+              <origin xyz="0 0 0" rpy="1.57 0 1.57" />
+              <geometry>
+                  <mesh filename="package://robile_description/meshes/sensors/UAM-05LPA.dae" scale="1 1 1" />
+              </geometry>
+          </visual>
+          <collision>
+              <origin xyz="0 0 0" rpy="1.57 0 1.57" />
+              <geometry>
+                  <mesh filename="package://robile_description/meshes/sensors/UAM-05LPA.dae" scale="1 1 1" />
+              </geometry>
+          </collision>
+      </link>
+      <xacro:gazebo_laser_plugin name="${name}" topic="${ros_topic}" sample_size="${sample_size}" update_rate="${update_rate}"
+                                  min_angle="${min_angle}" max_angle="${max_angle}" min_range="${min_range}" max_range="${max_range}"
+                                  visualize="${visualize}" sensor_type="gpu_lidar"/>
   </xacro:macro>
 </robot>

File: urdf/sensors/micro_scan.urdf.xacro (robot description, xacro)
@@ -1,30 +1,38 @@
 <?xml version="1.0"?>
-<robot xmlns:xacro="http://www.ros.org/wiki/xacro" name="kelo">
-  <xacro:macro name="sick_microscan3" params="name parent *origin ros_topic">
-    <joint name="${name}_joint" type="fixed">
-      <axis xyz="0 1 0" />
-      <xacro:insert_block name="origin" />
-      <parent link="${parent}"/>
-      <child link="${name}_link"/>
-    </joint>
-    <link name="${name}_link" type="laser">
-      <inertial>
-        <mass value="0.001" />
-        <origin xyz="0 0 0" rpy="0 0 0" />
-        <inertia ixx="0.0001" ixy="0" ixz="0" iyy="0.000001" iyz="0" izz="0.0001" />
-      </inertial>
-      <visual>
-        <origin xyz="0 0 -0.06" rpy="1.57 0 0" />
-      <geometry>
-        <mesh filename="package://robile_description/meshes/sensors/SICK-MICROSCAN3.dae" scale="0.001 0.001 0.001" />
-        </geometry>
-      </visual>
-      <collision>
-        <origin xyz="0 0 -0.06" rpy="1.57 0 0" />
-        <geometry>
-          <mesh filename="package://robile_description/meshes/sensors/SICK-MICROSCAN3.dae" scale="0.001 0.001 0.001" />
-        </geometry>
-      </collision>
-    </link>
-  </xacro:macro>
+<robot xmlns:xacro="http://www.ros.org/wiki/xacro">
+    <xacro:include filename="$(find robile_description)/urdf/sensors/common.xacro"/>
+    <xacro:macro name="sick_microscan3" params="*origin name:=base_laser_front
+                                          ros_topic parent:=base_link
+                                          sample_size:=540 update_rate:=10
+                                          min_angle:=-2.35619 max_angle:=2.35619
+                                          min_range:=0.1 max_range:=40.0 visualize:=true">
+        <joint name="${name}_joint" type="fixed">
+            <axis xyz="0 1 0" />
+            <xacro:insert_block name="origin" />
+            <parent link="${parent}"/>
+            <child link="${name}_link"/>
+        </joint>
+        <link name="${name}_link" type="laser">
+            <inertial>
+                <mass value="0.001" />
+                <origin xyz="0 0 0" rpy="0 0 0" />
+                <inertia ixx="0.0001" ixy="0" ixz="0" iyy="0.000001" iyz="0" izz="0.0001" />
+            </inertial>
+            <visual>
+                <origin xyz="0 0 -0.06" rpy="1.57 0 0" />
+                <geometry>
+                    <mesh filename="package://robile_description/meshes/sensors/SICK_MICROSCAN3.dae" scale="0.001 0.001 0.001" />
+                </geometry>
+            </visual>
+            <collision>
+                <origin xyz="0 0 -0.06" rpy="1.57 0 0" />
+                <geometry>
+                    <mesh filename="package://robile_description/meshes/sensors/SICK_MICROSCAN3.dae" scale="0.001 0.001 0.001" />
+                </geometry>
+            </collision>
+        </link>
+        <xacro:gazebo_laser_plugin name="${name}" topic="${ros_topic}" sample_size="${sample_size}" update_rate="${update_rate}"
+                                min_angle="${min_angle}" max_angle="${max_angle}" min_range="${min_range}" max_range="${max_range}"
+                                visualize="${visualize}" sensor_type="gpu_lidar"/>
+    </xacro:macro>
 </robot>
