Commit message: Fix wrong sensor file reference

File: urdf/sensors/micro_scan.urdf.xacro (robot description, xacro)
@@ -22,5 +22,5 @@
                 <origin xyz="0 0 -0.06" rpy="1.57 0 0" />
                 <geometry>
-                    <mesh filename="package://robile_description/meshes/sensors/SICK_MICROSCAN3.dae" scale="0.001 0.001 0.001" />
+                    <mesh filename="package://robile_description/meshes/sensors/SICK-MICROSCAN3.dae" scale="0.001 0.001 0.001" />
                 </geometry>
             </visual>
@@ -28,5 +28,5 @@
                 <origin xyz="0 0 -0.06" rpy="1.57 0 0" />
                 <geometry>
-                    <mesh filename="package://robile_description/meshes/sensors/SICK_MICROSCAN3.dae" scale="0.001 0.001 0.001" />
+                    <mesh filename="package://robile_description/meshes/sensors/SICK-MICROSCAN3.dae" scale="0.001 0.001 0.001" />
                 </geometry>
             </collision>
